File: ArduinoFlightController.kicad_pcb (KiCad board)
At the start: 4 copper layers, 40.5 x 40.5 mm, 45 parts, among them J1 USB_C_Receptacle_USB2.0, J2 PWM_PIN, J3 RC_IN, J4 Conn_01x02, J5 Conn_01x02, J6 Conn_01x02, J7 Conn_01x02, J8 Conn_01x02, SW1 NRST, U1 ATmega328P-A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

Commit message: add logo
Parts:
- added G***: LOGO, MyLogo:bit2byte_15m-x2mm, F.Cu at (120.8, 98.0)
- added G***: LOGO, MyLogo:Arrow_3mm-3mm, F.Cu at (138.7, 99.7)
- moved SW1 0.50 mm to (120.9, 107.9)
Routing:
- net /D5: track 8.60 -> 7.66 mm
- net /D6: track 9.86 -> 9.27 mm
- net /D4: track 16.0 -> 15.5 mm
